File: PiStormInside/PiStormInside_Full_Size_4_Layer.kicad_pcb (KiCad board)
At the start: 4 copper layers, 196.9 x 49 mm, 2 parts, among them CN0 Co-Processor, CN1 Co-Processor

Commit message: Updated from v1.0 to v1.1
Changed thermal reliefs as it was a bitch to solder them with (effectively) 3 ground planes.
Other:
- board text added: "Amiga 500 Internal Co-Processor adaptor v1.1 https://github.com/Fastdruid/AmigaHardware/ © David Sharp 2024"
- board text removed: "Amiga 500 Internal Co-Processor adaptor v1.0 https://github.com/Fastdruid/AmigaHardware/ © David Sharp 2024"
